File: MCU_Datalogger.kicad_pcb (KiCad board)
At the start: 2 copper layers, 50 x 30 mm, 29 parts, among them J1 Conn_01x04_Pin, J2 Conn_01x04_Pin, J3 Conn_01x09_Pin, J4 Conn_02x03_Odd_Even, U1 24LC1025, U2 DS1337S_, U3 24LC1025, U4 ATMEGA328P-AU, Y1 32.768 KHz, Y2 16 MHz

Commit message: Cleanup of layout
Routing:
- net GND: track 190.5 -> 57.0 mm, vias 5 -> 6
- net /Vcc: track 126.3 -> 52.6 mm, vias 7 -> 8
- net /RX: track 28.2 -> 35.9 mm, vias 1 -> 0
- net /TX: track 30.8 -> 38.3 mm, vias 1 -> 0
- net /MOSI: track 23.7 -> 30.0 mm, vias 0 -> 2
- net Net-(U4-PB7): track 30.5 -> 25.0 mm, vias 2 -> 3
- net /D2: track 29.3 -> 32.5 mm
- net /D7: track 19.0 -> 15.9 mm, vias 1 -> 0
- net /SDA: track 62.4 -> 59.3 mm, vias 2 -> 4
- net /D8: track 21.2 -> 18.2 mm, vias 1 -> 0
- net /RESET: track 27.0 -> 24.2 mm
- net /D6: track 17.4 -> 14.7 mm, vias 1 -> 0
- net Net-(U4-AREF): track 12.3 -> 14.5 mm
- net /D5: track 16.2 -> 14.4 mm, vias 1 -> 0
- net /MISO: track 19.2 -> 20.7 mm
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- added copper zone on In2.Cu, net /Vcc
- removed copper zone on B.Cu, net /Vcc
Other:
- copper layers 2 -> 4
- board text added: "4"
- board text removed: "0"
- board text removed: "0 mm"
- board text removed: "0.01 mm"
- board text removed: "0.02"
- board text removed: "0.035 mm"
- board text removed: "1"
- board text removed: "1.51 mm"
- board text removed: "2"
- board text removed: "3.3"
- board text removed: "4.5"
- board text removed: "B.Cu"
- board text removed: "B.Mask"
- board text removed: "B.Paste"
- board text removed: "B.Silkscreen"
- board text removed: "Bottom Silk Screen"
- board text removed: "Bottom Solder Mask"
- board text removed: "Bottom Solder Paste"
- board text removed: "Color"
- board text removed: "Dielectric"
- board text removed: "Epsilon R"
- board text removed: "F.Cu"
- board text removed: "F.Mask"
- board text removed: "F.Paste"
- board text removed: "F.Silkscreen"
- board text removed: "FR4"
- board text removed: "Layer Name"
- board text removed: "Loss Tangent"
- board text removed: "Material"
- board text removed: "Not specified"
- board text removed: "Thickness (mm)"
- board text removed: "Top Silk Screen"
- board text removed: "Top Solder Mask"
- board text removed: "Top Solder Paste"
- board text removed: "Type"
- board text removed: "copper"
- board text removed: "core"

Commit message: fixed pcb bug
Connections:
- J1 pad 4: /SCK -> /SCL
- R3 pad 2: /SCK -> /SCL
- U1 pad 6: /SCK -> /SCL
- U2 pad 6: /SCK -> /SCL
- U3 pad 6: /SCK -> /SCL
- U4 pad 28: /SCK -> /SCL
Routing:
- net /SCL: track 0.00 -> 86.3 mm, vias 0 -> 3
- net /SCK: track 94.0 -> 33.7 mm, vias 4 -> 1
